File: SLG46826G_実験評価用基板/回路図/src/20221225_SLG46826G.kicad_pcb (KiCad board)
At the start: 2 copper layers, 71.1 x 71.1 mm, 52 parts, among them IC1 SLG46826G, J1 GROVE-CONNECTOR-DIP_4P-2.0_, J2 Conn_01x20_Male, J3 Conn_01x20_Male, J4 Conn_01x15_Male, J5 Conn_01x15_Male, J6 Conn_01x15_Male, U1 MCP1703A-3302_SOT23

Commit message: update SLG46826G_実験評価用基板
Parts:
- R1, R10, R11, R12, R13, R14, R15, R16, R17, R2, R3, R4, R5, R6, R7, R8, R9: value 2k -> 1k
Connections:
- J1 pad 1: GND -> SCL
- J1 pad 2: VCC -> SDA
- J1 pad 3: SDA -> VCC
- J1 pad 4: SCL -> GND
Routing:
- net GND: track 325.8 -> 316.4 mm
- net (no net): vias 216 -> 0
Other:
- board text added: "Output LED Enabled"
- board text added: "PU/PD Setting"
- board text added: "VCC"
- board text removed: "5V"
- board text removed: "Conn_01x15_Male"
- board text removed: "LED Enabled"
