File: SLG46826G_実験評価用基板/回路図/src/20221225_SLG46826G.kicad_sch (KiCad schematic)
At the start: 52 parts, among them IC1 SLG46826G, J1 GROVE-CONNECTOR-DIP_4P-2.0_, J2 Conn_01x20_Male, J3 Conn_01x20_Male, J4 Conn_01x15_Male, J5 Conn_01x15_Male, J6 Conn_01x15_Male, U1 MCP1703A-3302_SOT23

Commit message: update SLG46826G_実験評価用基板
Parts:
- R1, R10, R11, R12, R13, R14, R15, R16, R17, R2, R3, R4, R5, R6, R7, R8, R9: value 2k -> 1k
Connections:
- net GND: now also J1.4; no longer J1.1
- net SCL: now also J1.1; no longer J1.4
- net SDA: now also J1.2; no longer J1.3
- net VCC: now also J1.3; no longer J1.2
Other:
- moved on the sheet: J1
